File: kicad/trailblazear.kicad_sch (KiCad schematic)
At the start: 7 parts, among them J1 USB_C_Receptacle

Commit message: updates
Parts:
- D1: footprint (none) -> Connector_PinHeader_2.54mm:PinHeader_1x04_P2.54mm_Vertical
- R1, R2, R3: footprint (none) -> Resistor_THT:R_Axial_DIN0207_L6.3mm_D2.5mm_P10.16mm_Horizontal
Changed lines of the file:
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@@
       (effects (font (size 2.54 2.54)) (justify right))
     )
-    (property "Footprint" "" (at 82.55 78.74 0)
+    (property "Footprint" "Resistor_THT:R_Axial_DIN0207_L6.3mm_D2.5mm_P10.16mm_Horizontal" (at 82.55 78.74 0)
       (effects (font (size 2.54 2.54)) hide)
     )
@@
       (effects (font (size 1.27 1.27)))
     )
-    (property "Footprint" "" (at 223.52 54.61 0)
+    (property "Footprint" "Connector_PinHeader_2.54mm:PinHeader_1x04_P2.54mm_Vertical" (at 223.52 54.61 0)
       (effects (font (size 1.27 1.27)) (justify left top) hide)
     )
@@
       (effects (font (size 2.54 2.54)))
     )
-    (property "Footprint" "" (at 196.85 46.99 0)
+    (property "Footprint" "Resistor_THT:R_Axial_DIN0207_L6.3mm_D2.5mm_P10.16mm_Horizontal" (at 196.85 46.99 0)
       (effects (font (size 2.54 2.54)) hide)
     )
@@
       (effects (font (size 2.54 2.54)) (justify right))
     )
-    (property "Footprint" "" (at 87.63 78.74 0)
-      (effects (font (size 2.54 2.54)) hide)
-    )
+    (property "Footprint" "Resistor_THT:R_Axial_DIN0207_L6.3mm_D2.5mm_P10.16mm_Horizontal" (at 87.63 78.74 0)
+      (effects (font (size 2.54 2.54)) hide)
+    )
